File: PCB Files/newpcb.kicad_pcb (KiCad board)
At the start: 2 copper layers, 0 parts

Commit message: Updated PCB, worked on radio section, positioned chips and stuff on board
Parts:
- added A1: Adafruit_Feather_Generic, Module:Adafruit_Feather, F.Cu at (106.8, 66.8)
- added C1: 100nF, Capacitor_SMD:C_0603_1608Metric_Pad1.08x0.95mm_HandSolder, F.Cu at (403.8, 132.4)
- added C11: 10nF, Capacitor_SMD:C_0603_1608Metric_Pad1.08x0.95mm_HandSolder, F.Cu at (403.8, 144.9)
- added C12: 100nF, Capacitor_SMD:C_0603_1608Metric_Pad1.08x0.95mm_HandSolder, F.Cu at (157.1, 38.5)
- added C13: 10nF, Capacitor_SMD:C_0603_1608Metric_Pad1.08x0.95mm_HandSolder, F.Cu at (408.2, 132.4)
- added C14: 100nF, Capacitor_SMD:C_0603_1608Metric_Pad1.08x0.95mm_HandSolder, F.Cu at (408.2, 134.9)
- added C15: 100nF, Capacitor_SMD:C_0603_1608Metric_Pad1.08x0.95mm_HandSolder, F.Cu at (408.2, 137.4)
- added C16: 100nF, Capacitor_SMD:C_0603_1608Metric_Pad1.08x0.95mm_HandSolder, F.Cu at (408.2, 139.9)
- added C17: 10nF, Capacitor_SMD:C_0603_1608Metric_Pad1.08x0.95mm_HandSolder, F.Cu at (158.6, 38.5)
- added C2: 100nF, Capacitor_SMD:C_0603_1608Metric_Pad1.08x0.95mm_HandSolder, F.Cu at (403.8, 134.9)
- added C3: 100nF, Capacitor_SMD:C_0603_1608Metric_Pad1.08x0.95mm_HandSolder, F.Cu at (403.8, 137.4)
- added C4: 10nF, Capacitor_SMD:C_0603_1608Metric_Pad1.08x0.95mm_HandSolder, F.Cu at (403.8, 139.9)
- added C5: 100nF, Capacitor_SMD:C_0603_1608Metric_Pad1.08x0.95mm_HandSolder, F.Cu at (403.8, 142.4)
- added D1: LED, LED_SMD:LED_0603_1608Metric_Pad1.05x0.95mm_HandSolder, F.Cu at (398.1, 89.1)
- added FB1: FerriteBead, Inductor_SMD:L_0603_1608Metric_Pad1.05x0.95mm_HandSolder, F.Cu at (161.0, 37.5)
- added J1: Conn_Coaxial, Connector_Coaxial:SMA_Molex_73251-1153_EdgeMount_Horizontal, F.Cu at (162.7, 25.8)
- added J2: Conn_Coaxial, Connector_Coaxial:SMA_Molex_73251-1153_EdgeMount_Horizontal, F.Cu at (136.3, 25.8)
- added J3: USB_C_Receptacle_USB2.0_16P, Connector_USB:USB_C_Receptacle_HRO_TYPE-C-31-M-12, F.Cu at (195.1, 102.9)
- added J4: Conn_Coaxial, Connector_Coaxial:U.FL_Molex_MCRF_73412-0110_Vertical, F.Cu at (196.7, 53.2)
- added J5: Conn_01x02(JST Vertical), Connector_JST:JST_PH_B2B-PH-K_1x02_P2.00mm_Vertical, F.Cu at (108.5, 39.5)
- added NT1: NetTie_2, NetTie:NetTie-2_SMD_Pad2.0mm, F.Cu at (104.0, 42.5)
- added R1: 10kO, Resistor_SMD:R_0603_1608Metric_Pad0.98x0.95mm_HandSolder, F.Cu at (408.2, 142.4)
- added R10: 470O, Resistor_SMD:R_0603_1608Metric_Pad0.98x0.95mm_HandSolder, F.Cu at (158.0, 36.0)
- added R11: 470O, Resistor_SMD:R_0603_1608Metric_Pad0.98x0.95mm_HandSolder, F.Cu at (158.0, 34.5)
- added R12: 470O, Resistor_SMD:R_0603_1608Metric_Pad0.98x0.95mm_HandSolder, F.Cu at (158.0, 33.0)
- added R13: 470O, Resistor_SMD:R_0603_1608Metric_Pad0.98x0.95mm_HandSolder, F.Cu at (158.0, 31.5)
- added R14: 470O, Resistor_SMD:R_0603_1608Metric_Pad0.98x0.95mm_HandSolder, F.Cu at (158.0, 30.0)
- added R15: 470O, Resistor_SMD:R_0603_1608Metric_Pad0.98x0.95mm_HandSolder, F.Cu at (158.0, 28.5)
- added R2: 5.1kO, Resistor_SMD:R_0603_1608Metric_Pad0.98x0.95mm_HandSolder, F.Cu at (408.2, 144.9)
- added R3: 5.1kO, Resistor_SMD:R_0603_1608Metric_Pad0.98x0.95mm_HandSolder, F.Cu at (408.2, 147.4)
- added R4: 1kO, Resistor_SMD:R_0603_1608Metric_Pad0.98x0.95mm_HandSolder, F.Cu at (412.5, 132.4)
- added R5: 1kO, Resistor_SMD:R_0603_1608Metric_Pad0.98x0.95mm_HandSolder, F.Cu at (412.5, 134.9)
- added R6: 2.2kO, Resistor_SMD:R_0603_1608Metric_Pad0.98x0.95mm_HandSolder, F.Cu at (412.5, 137.4)
- added R7: 2.2kO, Resistor_SMD:R_0603_1608Metric_Pad0.98x0.95mm_HandSolder, F.Cu at (412.5, 139.9)
- added R8: 470O, Resistor_SMD:R_0603_1608Metric_Pad0.98x0.95mm_HandSolder, F.Cu at (141.5, 37.0)
- added R9: 470O, Resistor_SMD:R_0603_1608Metric_Pad0.98x0.95mm_HandSolder, F.Cu at (141.5, 35.5)
- added SW1: Keyboard_6R13C, KeebDeck_Keyboard:Keyboard_6R13C, F.Cu at (149.8, 139.8)
- added SW2: SW_SPST(Battery Enable), Button_Switch_SMD:SW_DIP_SPSTx01_Slide_6.7x4.1mm_W6.73mm_P2.54mm_LowProfile_JPin, F.Cu at (114.5, 39.5)
- added SW3: SW_Push(Keyboard Boot), Button_Switch_SMD:SW_Push_1TS009xxxx-xxxx-xxxx_6x6x5mm, F.Cu at (357.0, 131.0)
- added SW4: SW_Push(Feather Reset), Button_Switch_SMD:SW_Push_1TS009xxxx-xxxx-xxxx_6x6x5mm, F.Cu at (336.0, 147.0)
- added U1: Wio-LR2021, Footprint and Symbol Library:Wio-LR2021_V1, F.Cu at (148.8, 18.9)
- added U2: MCP23017x-x-SP, Package_DIP:DIP-28_W7.62mm, F.Cu at (110.8, 74.3)
- added U3: STM32F042C4Ux, Package_DFN_QFN:QFN-48-1EP_7x7mm_P0.5mm_EP5.6x5.6mm, B.Cu at (104.9, 108.9)
- added U4: CR2013-MI2120, Display:CR2013-MI2120, F.Cu at (187.0, 100.2)
- added U5: TMP100, Package_TO_SOT_SMD:SOT-23-6, F.Cu at (158.7, 56.6)
- added U7: 790, footprints:PA1616S_ADA, F.Cu at (189.7, 42.2)
- added U8: MPU-9250, Sensor_Motion:InvenSense_QFN-24_3x3mm_P0.4mm, F.Cu at (158.7, 49.0)
Routing:
- net /R.5: track 0.00 -> 79.2 mm
- net /R.4: track 0.00 -> 79.2 mm
- net /R.3: track 0.00 -> 79.2 mm
- net /R.2: track 0.00 -> 79.2 mm
- net /R.1: track 0.00 -> 79.2 mm
- net /R.0: track 0.00 -> 76.1 mm
- net /SCK: track 0.00 -> 51.3 mm, vias 0 -> 1
- net /RX: track 0.00 -> 50.5 mm, vias 0 -> 1
- net /MOSI: track 0.00 -> 48.2 mm, vias 0 -> 1
- net /TX: track 0.00 -> 47.9 mm, vias 0 -> 1
- net Net-(U3-PB1): track 0.00 -> 44.1 mm
- net /MISO: track 0.00 -> 43.4 mm, vias 0 -> 1
- net Net-(U3-PB2): track 0.00 -> 43.2 mm
- net Net-(U3-PB11): track 0.00 -> 42.2 mm
- net Net-(U3-PB10): track 0.00 -> 40.9 mm
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- added copper zone on In2.Cu, net +3V3
- added copper zone on F.Cu, net GND
- added copper zone on In1.Cu, net GND
- added copper zone on In2.Cu, net RF+3V3
Other:
- board outline added: 99.5 x 150 mm
- copper layers 2 -> 4

Commit message: Finished keyboard controller matrix, did some wiring
Parts:
- U3: moved to F.Cu
- moved R2 305.9 mm to (107.0, 91.5), turned to 90 degrees
- moved R3 304.8 mm to (108.5, 91.5), turned to 90 degrees
- moved SW3 256.0 mm to (105.0, 86.0), turned to 180 degrees
- moved R4 253.9 mm to (175.4, 41.5)
- moved SW4 242.3 mm to (105.0, 74.0)
- moved D1 224.3 mm to (178.8, 41.5)
- moved J3 91.2 mm to (104.0, 98.5), turned to -90 degrees
- moved C1 0.18 mm to (404.0, 132.4)
- turned U3 to 0 degrees
Connections:
- net /R.3 renamed /R3
- net /R.4 renamed /R4
- net /R.5 renamed /R5
- net Net-(U3-PB0) renamed /C0
- net Net-(U3-PB1) renamed /C1
- SW1 pad C10: Net-(U3-PB10) -> /C10
- SW1 pad C11: Net-(U3-PB11) -> /C11
- SW1 pad C12: Net-(U3-PB12) -> /C12
- SW1 pad C2: Net-(U3-PB3) -> /C2
- SW1 pad C3: Net-(U3-PB4) -> /C3
- SW1 pad C4: Net-(U3-PB2) -> /C4
- SW1 pad C5: Net-(U3-PB5) -> /C5
- SW1 pad C6: Net-(U3-PB6) -> /C6
- SW1 pad C7: Net-(U3-PB7) -> /C7
- SW1 pad C8: Net-(U3-PB9) -> /C8
- SW1 pad C9: Net-(U3-PB8) -> /C9
- SW1 pad R0: /R.0 -> /R0
- SW1 pad R1: /R.1 -> /R1
- SW1 pad R2: /R.2 -> /R2
- U3 pad 10: /R.0 -> unconnected-(U3-PA0-Pad10)
- U3 pad 11: /R.1 -> unconnected-(U3-PA1-Pad11)
- U3 pad 12: /R.2 -> /R0
- U3 pad 16: unconnected-(U3-PA6-Pad16) -> /R2
- U3 pad 17: unconnected-(U3-PA7-Pad17) -> /R1
- U3 pad 20: Net-(U3-PB2) -> /C2
- U3 pad 21: Net-(U3-PB10) -> /C3
- U3 pad 22: Net-(U3-PB11) -> /C4
- U3 pad 25: Net-(U3-PB12) -> /C5
- U3 pad 26: unconnected-(U3-PB13-Pad26) -> /C6
- U3 pad 27: unconnected-(U3-PB14-Pad27) -> /C7
- U3 pad 28: unconnected-(U3-PB15-Pad28) -> /C8
- U3 pad 39: Net-(U3-PB3) -> unconnected-(U3-PB3-Pad39)
- U3 pad 40: Net-(U3-PB4) -> unconnected-(U3-PB4-Pad40)
- U3 pad 41: Net-(U3-PB5) -> unconnected-(U3-PB5-Pad41)
- U3 pad 42: Net-(U3-PB6) -> /C12
- U3 pad 43: Net-(U3-PB7) -> /C11
- U3 pad 45: Net-(U3-PB8) -> /C10
- U3 pad 46: Net-(U3-PB9) -> /C9
Routing:
- net /C12: track 0.00 -> 133.6 mm, vias 0 -> 1
- net /C11: track 0.00 -> 132.9 mm, vias 0 -> 2
- net /C10: track 0.00 -> 124.8 mm, vias 0 -> 2
- net /C9: track 0.00 -> 113.3 mm, vias 0 -> 2
- net /R2: track 0.00 -> 102.9 mm
- net /C7: track 0.00 -> 94.8 mm, vias 0 -> 1
- net /R1: track 0.00 -> 94.8 mm
- net /C8: track 0.00 -> 90.0 mm, vias 0 -> 1
- net /R0: track 0.00 -> 88.5 mm, vias 0 -> 2
- net /C6: track 0.00 -> 86.1 mm, vias 0 -> 1
- net /C4: track 0.00 -> 81.9 mm, vias 0 -> 1
- net /R.2: track 79.2 -> 0.00 mm
- net /R.1: track 79.2 -> 0.00 mm
- net /R.0: track 76.1 -> 0.00 mm
- net /C5: track 0.00 -> 71.8 mm, vias 0 -> 1
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Other:
- board size 99.5 x 150 mm -> 99.5 x 150.5 mm

Commit message: Finish PCB, yay
Parts:
- removed C13: 10nF, Capacitor_SMD:C_0603_1608Metric_Pad1.08x0.95mm_HandSolder
- removed C14, C15: 100nF, Capacitor_SMD:C_0603_1608Metric_Pad1.08x0.95mm_HandSolder
- removed U8: MPU-9250, Sensor_Motion:InvenSense_QFN-24_3x3mm_P0.4mm
- added C6: 220nF, Capacitor_SMD:C_0603_1608Metric_Pad1.08x0.95mm_HandSolder, F.Cu at (158.4, 51.6)
- added C7: 100nF, Capacitor_SMD:C_0603_1608Metric_Pad1.08x0.95mm_HandSolder, F.Cu at (160.6, 47.5)
- added C8: 10nF, Capacitor_SMD:C_0603_1608Metric_Pad1.08x0.95mm_HandSolder, F.Cu at (162.1, 47.5)
- added C9: 100nF, Capacitor_SMD:C_0603_1608Metric_Pad1.08x0.95mm_HandSolder, F.Cu at (159.0, 45.6)
- added U6: LSM303AGR, LSM303AGR:PQFN50P200X200X100-12N, F.Cu at (158.5, 48.8)
- C1, C16, C2, C3, C4, C5: moved to B.Cu
- moved R5 316.8 mm to (102.5, 69.5)
- moved R1 310.1 mm to (102.5, 90.5)
- moved C1 303.7 mm to (101.3, 107.5), turned to -90 degrees
- moved C4 302.8 mm to (102.5, 110.0)
- moved C3 302.5 mm to (102.8, 107.5), turned to -90 degrees
- moved C5 298.8 mm to (107.5, 104.0), turned to 180 degrees
- moved C2 296.7 mm to (108.0, 112.5), turned to 180 degrees
- moved C16 288.1 mm to (126.4, 80.0)
- moved R7 275.3 mm to (152.5, 49.5), turned to 90 degrees
- moved R6 272.3 mm to (152.5, 56.5), turned to 90 degrees
- moved C11 257.0 mm to (162.0, 58.0), turned to -90 degrees
- moved U4 67.1 mm to (123.0, 79.8), turned to 0 degrees
- moved SW1 0.50 mm to (150.3, 139.8)
Connections:
- U2 pad 26: /GPS.1PPS -> /INT_1_XL
- U2 pad 27: unconnected-(U2-GPA6-Pad27) -> /INT_2_XL
- U2 pad 28: unconnected-(U2-GPA7-Pad28) -> /INT_MAG/DRDY
- U7 pad 13: /GPS.1PPS -> unconnected-(U7-1PPS-Pad13)
Routing:
- net /SCL: track 0.20 -> 108.1 mm, vias 0 -> 2
- net /SDA: track 0.00 -> 102.4 mm
- net /GPS.RESET: track 0.00 -> 98.8 mm, vias 0 -> 1
- net /INT_1_XL: track 0.00 -> 59.2 mm, vias 0 -> 3
- net /P.RESET: track 0.00 -> 57.4 mm
- net /INT_MAG/DRDY: track 0.00 -> 57.4 mm, vias 0 -> 2
- net /INT_2_XL: track 0.00 -> 56.7 mm, vias 0 -> 2
- net /SC.D/C: track 0.00 -> 45.6 mm
- net /SC.MISO: track 0.00 -> 36.8 mm
- net /P.INTB: track 0.00 -> 32.0 mm
- net /SC.CLK: track 0.00 -> 31.0 mm
- net /P.INTA: track 0.00 -> 30.3 mm
- net /K.RESET: track 0.00 -> 29.8 mm, vias 0 -> 1
- net /SC.MOSI: track 0.00 -> 27.4 mm
- net +3V3: track 0.00 -> 26.2 mm, vias 3 -> 13
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
Commit message: fix error in gps uart
Connections:
- U7 pad 10: /RX -> /TX
- U7 pad 9: /TX -> /RX
Routing:
- net /TX: track 47.9 -> 46.9 mm
Changed lines of the file:
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@@
 			(size 2.0066 0.9906)
 			(layers "F.Cu" "F.Mask" "F.Paste")
-			(net "/TX")
+			(net "/RX")
 			(pinfunction "TX0_9")
 			(pintype "output")
@@
 			(size 2.0066 0.9906)
 			(layers "F.Cu" "F.Mask" "F.Paste")
-			(net "/RX")
+			(net "/TX")
 			(pinfunction "RX0_10")
 			(pintype "input")
@@
 	)
 	(segment
+		(start 158.25 49.495)
+		(end 158.25 50.5875)
+		(width 0.2)
+		(layer "F.Cu")
+		(net "Net-(U6-C1)")
+	)
+	(segment
+		(start 158.25 50.5875)
+		(end 158.45 50.7875)
+		(width 0.2)
+		(layer "F.Cu")
+		(net "Net-(U6-C1)")
+	)
+	(segment
 		(start 177.975 41.55)
 		(end 176.3 41.55)
@@
 	)
 	(via
-		(at 181.9 48.999998)
+		(at 181.9 47.499999)
 		(size 0.6)
 		(drill 0.3)
@@
 	)
 	(segment
-		(start 141.16 68.12)
-		(end 162.779998 68.12)
+		(start 150.1885 56.4915)
+		(end 139.86 66.82)
 		(width 0.2)
 		(layer "B.Cu")
@@
 	)
 	(segment
-		(start 139.86 66.82)
-		(end 141.16 68.12)
+		(start 172.908499 56.4915)
+		(end 150.1885 56.4915)
 		(width 0.2)
 		(layer "B.Cu")
@@
 	)
 	(segment
-		(start 162.779998 68.12)
-		(end 181.9 48.999998)
+		(start 181.9 47.499999)
+		(end 172.908499 56.4915)
 		(width 0.2)
 		(layer "B.Cu")
@@
 	)
 	(via
-		(at 181.9 47.499999)
+		(at 181.9 48.999998)
 		(size 0.6)
 		(drill 0.3)
@@
 	)
 	(segment
-		(start 142.4 66.82)
-		(end 144.72 64.5)
-		(width 0.2)
-		(layer "B.Cu")
-		(net "/TX")
-	)
-	(segment
-		(start 144.72 64.5)
-		(end 165.5 64.5)
+		(start 150.22 59)
+		(end 142.4 66.82)
 		(width 0.2)
 		(layer "B.Cu")
@@
 	)
 	(segment
-		(start 165.5 64.5)
-		(end 181.9 48.1)
+		(start 181.9 48.999998)
+		(end 171.899998 59)
 		(width 0.2)
 		(layer "B.Cu")
@@
 	)
 	(segment
-		(start 181.9 48.1)
-		(end 181.9 47.499999)
+		(start 171.899998 59)
+		(end 150.22 59)
 		(width 0.2)
 		(layer "B.Cu")
@@
 	)
 	(segment
-		(start 196.725 51.749999)
-		(end 196.725 49.774998)
-		(width 0.2)
-		(layer "F.Cu")
-		(net "Net-(J4-In)")
-	)
-	(segment
-		(start 196.725 49.774998)
-		(end 197.5 48.999998)
-		(width 0.2)
-		(layer "F.Cu")
-		(net "Net-(J4-In)")
-	)
-	(segment
 		(start 158.25 47.2)
 		(end 158.175 47.125)
@@
 	)
 	(segment
-		(start 158.25 49.495)
-		(end 158.25 50.5875)
+		(start 196.725 51.749999)
+		(end 196.725 49.774998)
 		(width 0.2)
 		(layer "F.Cu")
-		(net "Net-(U6-C1)")
+		(net "Net-(J4-In)")
 	)
 	(segment
-		(start 158.25 50.5875)
-		(end 158.45 50.7875)
+		(start 196.725 49.774998)
+		(end 197.5 48.999998)
 		(width 0.2)
 		(layer "F.Cu")
-		(net "Net-(U6-C1)")
+		(net "Net-(J4-In)")
 	)
 	(zone
